File: tackle_sensor_hardware.kicad_pcb (KiCad board)
At the start: 4 copper layers, 47 x 59.7 mm, 79 parts, among them J1 Conn_ARM_JTAG_SWD_10, J2 Conn_01x02_Male, J4 Conn_01x04_Male, J5 Conn_01x06_Male, Q1 DMP4051LK3, Q2 NCE0110K, SW1 PTS645SL43SMTR92 LFS, T1 DRQ125-330-R, U1 STM32G031Fx, U2 LM3488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

Commit message: REV2.1_UPLOAD
Parts:
- D4: value CLV1A-FKB-CK1VW1DE1BB7C3C3 -> MHPA3528RGBCT; footprint LED_SMD:LED_Cree-PLCC4_3.2x2.8mm_CCW -> rfc_footprint_lib:LED-ARRAY-SMD_4P-L3.5-W2.8-TL
- R15, R17, R19: value 0,0.5W -> 100,0.5W
- S1: value DS01-254-L-02BE -> DSWB02LHGET; footprint rfc_footprint_lib:SW_DS01-254-L-02BE -> rfc_footprint_lib:SW-TH_DSWB02LHGET
- turned D4 to 180 degrees
Connections:
- D4 pad 1: Net-(D4-Pad1) -> +12V
- D4 pad 2: +12V -> Net-(D4---Pad2)
- D4 pad 3: Net-(D4-Pad3) -> Net-(D4---Pad3)
- D4 pad 4: Net-(D4-Pad4) -> Net-(D4---Pad4)
- R11 pad 1: Net-(D4-Pad1) -> Net-(D4---Pad4)
- R13 pad 1: Net-(D4-Pad4) -> Net-(D4---Pad3)
- R14 pad 1: Net-(D4-Pad3) -> Net-(D4---Pad2)
Routing:
- net Net-(D4-Pad1): track 9.37 -> 0.00 mm
- net Net-(D4---Pad3): track 0.00 -> 5.94 mm
- net Net-(D4---Pad4): track 0.00 -> 4.91 mm
- net Net-(D4---Pad2): track 0.00 -> 4.69 mm
- net Net-(D4-Pad4): track 4.30 -> 0.00 mm
- net Net-(D4-Pad3): track 3.18 -> 0.00 mm
Other:
- board text added: "Tackle Sensor V4 REV2.1 5/23/2026"
- board text removed: "Tackle Sensor V4 REV2 2/4/2024"
