File: tackle_sensor_hardware.kicad_sch (KiCad schematic)
At the start: 77 parts, among them J1 Conn_ARM_JTAG_SWD_10, J2 Conn_01x02_Male, J4 Conn_01x04_Male, J5 Conn_01x06_Male, Q1 DMP4051LK3, Q2 NCE0110K, SW1 PTS645SL43SMTR92 LFS, T1 DRQ125-330-R, U1 STM32G031Fx, U2 LM3488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

Commit message: REV2.1_UPLOAD
Parts:
- removed D4: CLV1A-FKB-CK1VW1DE1BB7C3C3, LED_SMD:LED_Cree-PLCC4_3.2x2.8mm_CCW, symbol rfc_symbol_lib:CLV1A-FKB-CK1VW1DE1BB7C3C3
- removed S1: DS01-254-L-02BE, rfc_footprint_lib:SW_DS01-254-L-02BE, symbol DS01-254-L-02BE:DS01-254-L-02BE
- added D4: MHPA3528RGBCT, rfc_footprint_lib:LED-ARRAY-SMD_4P-L3.5-W2.8-TL, symbol rfc_symbol_lib:MHPA3528RGBCT
- added S1: DSWB02LHGET, rfc_footprint_lib:SW-TH_DSWB02LHGET, symbol rfc_symbol_lib:DSWB02LHGET
- C1, C13, C14, C3, C4, C9: JCSC_U (none) -> x; JLCPN C49678 -> C5137467
- C10, C11, C7: JCSC_U (none) -> x; JLCPN C90540 -> C5199872
- C12: JCSC_U (none) -> x; JLCPN C215761 -> C51953338
- C15, C2: JCSC_U (none) -> x; JLCPN C308830 -> C128459
- C5: JCSC_U (none) -> x; JLCPN C338130 -> C915853
- C6, J2, J4, Q1, Q2, R2, U1, U2, U4, U5: JCSC_U (none) -> x
- C8: JCSC_U (none) -> x; JLCPN C1523 -> C106205
- D1: JCSC_U (none) -> x; JLCPN C188533 -> C2932746
- D2: symbol rfc_symbol_lib:SS2PH10HM3_A/H -> rfc_symbol_lib:SS2PH10HM3_A/H; JCSC_U (none) -> x; JLCPN C41029 -> C727076
- D3: JCSC_U (none) -> x; JLCPN C72038 -> C84268
- F1: JCSC_U (none) -> x; JLCPN C207046 -> C70097
- FID1, FID2, FID3, H1, H2, H3, H4, TP1, TP10, TP11, TP12, TP13, TP14, TP15, TP2, TP3, TP8, TP9: JCSC_U (none) -> x; now left out of the parts list
- J1: JCSC_U (none) -> x; JLCPN C150517 -> C41376037
- J5: JCSC_U (none) -> x; JLCPN (none) -> C144397
- R1, R10, R21, R23, R3, R9: JCSC_U (none) -> x; JLCPN C25744 -> C2906861
- R11, R12, R13, R14: JCSC_U (none) -> x; JLCPN C21190 -> C2907002
- R15, R17, R19: value 0,0.5W -> 100,0.5W; JCSC_U (none) -> x
- R16, R18, R20, R24, R25: JCSC_U (none) -> x; JLCPN C25091 -> C2909336
- R22, R5: JCSC_U (none) -> x; JLCPN (none) -> C2906859
- R4: JCSC_U (none) -> x; JLCPN C54968 -> C5126096
- R6: JCSC_U (none) -> x; JLCPN C25076 -> C2906860
- R8: JCSC_U (none) -> x; JLCPN C100545 -> C2998184
- SW1: JCSC_U (none) -> x; JLCPN C221875 -> C7470150
- T1: JLCPN (none) -> C3273455
- U3: JCSC_U (none) -> x; JLCPN C155639 -> C189624
Connections:
- net +12V: now also D4.1 (-)
- net ELIGIBLE_SELECT: now also S1.1
- net HOME_SELECT: now also S1.2
- net at R23.1: now also S1.4
- net at R21.1: now also S1.3
- net at R11.1: now also D4.4 (-)
- net at R14.1: now also D4.2 (-)
- net at R13.1: now also D4.3 (-)
Other:
- note added: "CHANGE ME"
- note added: "TODO: - Change R7 (follow schematic?) - Find inductor that will work OR order parts to JLCPCB"
- moved on the sheet: R11, R14, R23
